File: domino-tile-pcb/domino-tile-pcb.kicad_sch (KiCad schematic)
At the start: 2 parts, among them J1 Conn_02x11_Odd_Even

Commit message: do more things
Parts:
- removed J1: Conn_02x11_Odd_Even, symbol Connector_Generic:Conn_02x11_Odd_Even
- added D10, D11, D12, D2, D3, D4, D5, D6, D7, D8, D9: ~, LED_SMD:LED_PLCC_2835_Handsoldering, symbol Device:LED
- added J1: ~, Connector_IDC:IDC-Header_2x06_P2.54mm_Vertical_SMD, symbol Connector_Generic:Conn_02x06_Odd_Even
- added J2: ~, Connector_JST:JST_EH_B3B-EH-A_1x03_P2.50mm_Vertical, symbol Connector:Conn_01x03_Pin
- added JP1, JP10, JP11, JP12, JP2, JP3, JP4, JP5, JP6, JP7, JP8, JP9: ~, Jumper:SolderJumper-2_P1.3mm_Open_Pad1.0x1.5mm, symbol Jumper:Jumper_2_Open
- added R1, R10, R11, R12, R2, R3, R4, R5, R6, R7, R8, R9: 470, Resistor_SMD:R_0805_2012Metric_Pad1.20x1.40mm_HandSolder, symbol Device:R
- D1: value LED -> ~; footprint (none) -> LED_SMD:LED_PLCC_2835_Handsoldering
Connections:
- net at D1.1 (K): now also JP1.1 (A), R1.1
- net at D1.2 (A): now also J1.4 (Pin_4), JP1.2 (B)
- new net: D12.1 (K), JP12.1 (A), R12.1
- new net: D12.2 (A), J1.9 (Pin_9), JP12.2 (B)
- new net: D2.1 (K), JP2.1 (A), R2.1
- new net: D2.2 (A), J1.2 (Pin_2), JP2.2 (B)
- new net: D6.1 (K), JP6.1 (A), R6.1
- new net: D9.1 (K), JP9.1 (A), R9.1
- new net: D9.2 (A), J1.10 (Pin_10), JP9.2 (B)
- new net: D3.1 (K), JP3.1 (A), R3.1
- new net: D3.2 (A), J1.1 (Pin_1), JP3.2 (B)
- new net: D7.1 (K), JP7.1 (A), R7.1
- new net: D7.2 (A), J1.7 (Pin_7), JP7.2 (B)
- new net: D11.2 (A), J1.11 (Pin_11), JP11.2 (B)
- new net: D10.2 (A), J1.12 (Pin_12), JP10.2 (B)
- new net: D4.2 (A), J1.3 (Pin_3), JP4.2 (B)
- new net: D8.2 (A), J1.5 (Pin_5), JP8.2 (B)
- new net: D6.2 (A), J1.6 (Pin_6), JP6.2 (B)
- new net: D5.2 (A), J1.8 (Pin_8), JP5.2 (B)
- new net: D5.1 (K), JP5.1 (A), R5.1
- new net: D8.1 (K), JP8.1 (A), R8.1
- new net: D10.1 (K), JP10.1 (A), R10.1
- new net: D11.1 (K), JP11.1 (A), R11.1
- new net: D4.1 (K), JP4.1 (A), R4.1
- new net GND: J2.2 (Pin_2), R1.2, R10.2, R11.2, R12.2, R2.2, R3.2, R4.2, R5.2, R6.2, R7.2, R8.2, R9.2
